File: pcb/current-sense/current-sense.kicad_pcb (KiCad board)
At the start: 4 copper layers, 130 x 25 mm, 113 parts, among them J1 M3, J2 M3, J3 Tag Connect, J4 M3, J5 M3, J6 Conn_Coaxial, J7 AA Holder, J8 DNP, Q1 FDC6327C, SW1 SW_Push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

Commit message: fix for drc
Routing:
- net GNDREF: track 18.7 -> 20.3 mm
Changed lines of the file:
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@@
-	)
-	(segment
-		(start -26.3398 -38.3286)
-		(end -26.289 -38.3286)
-		(width 0.127)
-		(layer "In1.Cu")
-		(net "")
-	)
-	(segment
-		(start -26.289 -38.3286)
-		(end -26.2636 -38.354)
-		(width 0.127)
-		(layer "In1.Cu")
-		(net "")
 	)
 	(segment
@@
 	)
 	(segment
+		(start -26.54 -38.34)
+		(end -26.34 -38.34)
+		(width 0.16)
+		(layer "In1.Cu")
+		(net "GNDREF")
+	)
+	(segment
 		(start -26.75 -39.5)
 		(end -25.75 -39.5)
@@
 	)
 	(segment
+		(start -26.3 -38.38)
+		(end -26.18 -38.38)
+		(width 0.16)
+		(layer "In1.Cu")
+		(net "GNDREF")
+	)
+	(segment
+		(start -26.75 -38.55)
+		(end -26.54 -38.34)
+		(width 0.16)
+		(layer "In1.Cu")
+		(net "GNDREF")
+	)
+	(segment
+		(start -26.75 -39.5)
+		(end -26.75 -38.55)
+		(width 0.16)
+		(layer "In1.Cu")
+		(net "GNDREF")
+	)
+	(segment
 		(start -26.2636 -35.687)
 		(end -26.3398 -35.6108)
@@
 		(layer "In1.Cu")
 		(net "GNDREF")
+	)
+	(segment
+		(start -26.34 -38.34)
+		(end -26.3 -38.38)
+		(width 0.16)
+		(layer "In1.Cu")
+		(net "GNDREF")
